File: pcb/ece477.sch (KiCad schematic (older format))
At the start: 16 parts, among them J1 USB_B, SW1 SW_DIP_x01, U1 ESP32-WROOM-32, U2 FT232RL-REEL, U3 LM3671, U4 ADA254, U5 ADA751

Commit message: shifted LM3671 to top right
Parts:
- removed FB1: Ferrite_Bead, Ferrite_THT:LairdTech_28C0236-0JW-10, symbol Device:Ferrite_Bead
- added C6: 10uF, Capacitor_SMD:CP_Elec_3x5.3, symbol Device:CP
- added D1, D2: LED, LED_SMD:LED_0201_0603Metric, symbol Device:LED
- added R2: 100kΩ, Resistor_SMD:R_0201_0603Metric, symbol Device:R
- added R3, R4: 1kΩ, Resistor_SMD:R_0201_0603Metric, symbol Device:R
- C4: value 100nF -> 0.1uF
- C5: value 10nF -> 0.1uF
Connections:
- net GND: now also C6.2
- net at C2.2, L1.1, R1.1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: no longer U2.20 (VCC)
- net at C3.2, SW1.2, U3.1 (Vin)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: now also R2.2; no longer U3.3 (EN)
- net at C5.1, J1.1 (VBUS): now also U2.20 (VCC), C6.1, R3.1, R4.1
- net at U2.22 (CBUS1): now also D2.1 (K)
- net at U2.23 (CBUS0): now also D1.1 (K)
- new net: R2.1, U3.3 (EN)
- new net: D1.2 (A), R3.2
- new net: D2.2 (A), R4.2
Changed lines of the file:
@@
 Wire Wire Line
 	7300 4550 7150 4550
-Connection ~ 7300 3550
 $Comp
 L power:GND #PWR0101
@@
 	6050 5650 6050 6050
 Connection ~ 6050 6050
-Wire Wire Line
-	5250 3600 5750 3600
 Wire Wire Line
 	5250 3800 6800 3800
@@
 	5050 2450 6350 2450
 Wire Wire Line
-	6350 2450 6350 2150
-Wire Wire Line
 	6350 2150 6250 2150
 Connection ~ 5050 2450
 Wire Wire Line
 	5050 2450 5050 1950
-Wire Wire Line
-	6250 2050 6350 2050
-Wire Wire Line
-	6350 2050 6350 2150
-Connection ~ 6350 2150
 $Comp
 L Device:C C3
@@
 F 3 "~" H 6350 1700 50  0001 C CNN
 	1    6350 1700
-	1    0    0    -1
-$EndComp
-Wire Wire Line
-	6350 1850 6350 2050
-Connection ~ 6350 2050
-$Comp
-L Device:C C4
-U 1 1 5F7A38A5
-P 7100 3000
-F 0 "C4" H 7215 3046 50  0000 L CNN
-F 1 "100nF" H 7215 2955 50  0000 L CNN
-F 2 "Capacitor_SMD:C_0201_0603Metric" H 7138 2850 50  0001 C CNN
-F 3 "~" H 7100 3000 50  0001 C CNN
-	1    7100 3000
-	-1   0    0    1
-$EndComp
-$Comp
-L power:GND #PWR0103
-U 1 1 5F7A3D3E
-P 7100 3150
-F 0 "#PWR0103" H 7100 2900 50  0001 C CNN
-F 1 "GND" H 7105 2977 50  0000 C CNN
-F 2 "" H 7100 3150 50  0001 C CNN
-F 3 "" H 7100 3150 50  0001 C CNN
-	1    7100 3150
 	1    0    0    -1
 $EndComp
@@
 	-1   0    0    1
 $EndComp
-Wire Wire Line
-	8600 1950 8700 1950
+Connection ~ 9000 1550
+Wire Wire Line
+	9000 1250 9500 1250
+Wire Wire Line
+	9500 1250 9500 2350
+Wire Wire Line
+	8700 2350 8700 2150
+Wire Wire Line
+	7700 3550 7700 3850
+Wire Wire Line
+	5950 1550 6350 1550
+Connection ~ 6350 1550
+Wire Wire Line
+	8300 2650 8200 2650
+Wire Wire Line
+	6800 2650 6800 3800
+Wire Wire Line
+	3600 1550 5400 1550
+Wire Wire Line
+	6050 6050 4850 6050
+Wire Wire Line
+	4850 6050 4850 6100
+Wire Wire Line
+	4850 6100 4650 6100
+$Comp
+L Device:R R2
+U 1 1 5F815B5C
+P 6650 2100
+F 0 "R2" H 6720 2146 50  0000 L CNN
+F 1 "100kΩ" H 6720 2055 50  0000 L CNN
+F 2 "Resistor_SMD:R_0201_0603Metric" V 6580 2100 50  0001 C CNN
+F 3 "~" H 6650 2100 50  0001 C CNN
+	1    6650 2100
+	1    0    0    -1
+$EndComp
+Wire Wire Line
+	5250 3600 5750 3600
+Wire Wire Line
+	5750 3950 5750 3600
+Wire Wire Line
+	5750 3950 8300 3950
+$Comp
+L power:GND #PWR0103
+U 1 1 5F7A3D3E
+P 7100 3150
+F 0 "#PWR0103" H 7100 2900 50  0001 C CNN
+F 1 "GND" H 7105 2977 50  0000 C CNN
+F 2 "" H 7100 3150 50  0001 C CNN
+F 3 "" H 7100 3150 50  0001 C CNN
+	1    7100 3150
+	1    0    0    -1
+$EndComp
+Wire Wire Line
+	7700 3850 8950 3850
+$Comp
+L Device:C C4
+U 1 1 5F7A38A5
+P 7100 3000
+F 0 "C4" H 7215 3046 50  0000 L CNN
+F 1 "0.1uF" H 7215 2955 50  0000 L CNN
+F 2 "Capacitor_SMD:C_0201_0603Metric" H 7138 2850 50  0001 C CNN
+F 3 "~" H 7100 3000 50  0001 C CNN
+	1    7100 3000
+	-1   0    0    1
+$EndComp
 $Comp
 L Device:C C5
@@
 P 9000 1400
 F 0 "C5" H 9115 1446 50  0000 L CNN
-F 1 "10nF" H 9115 1355 50  0000 L CNN
+F 1 "0.1uF" H 9115 1355 50  0000 L CNN
 F 2 "Capacitor_SMD:C_0201_0603Metric" H 9038 1250 50  0001 C CNN
 F 3 "~" H 9000 1400 50  0001 C CNN
@@
 	1    0    0    -1
 $EndComp
-Connection ~ 9000 1550
-Wire Wire Line
-	9000 1250 9500 1250
-Wire Wire Line
-	9500 1250 9500 2350
-Wire Wire Line
-	9500 2350 8950 2350
-Wire Wire Line
-	8700 2350 8700 2150
-$Comp
-L Device:Ferrite_Bead FB1
-U 1 1 5F7C0CC2
-P 8950 2500
-F 0 "FB1" H 9087 2546 50  0000 L CNN
-F 1 "Ferrite_Bead" H 9087 2455 50  0000 L CNN
-F 2 "Ferrite_THT:LairdTech_28C0236-0JW-10" V 8880 2500 50  0001 C CNN
-F 3 "~" H 8950 2500 50  0001 C CNN
-	1    8950 2500
-	1    0    0    -1
-$EndComp
-Connection ~ 8950 2350
-Wire Wire Line
-	8950 2350 8700 2350
-Wire Wire Line
-	7700 3550 7700 3850
-Wire Wire Line
-	7700 3850 8950 3850
-Wire Wire Line
-	8950 3850 8950 2650
-Wire Wire Line
-	5950 1550 6350 1550
-Connection ~ 6350 1550
+Wire Wire Line
+	8200 2950 8350 2950
+Wire Wire Line
+	8300 3950 8300 2650
+Wire Wire Line
+	8600 1950 8700 1950
+Wire Wire Line
+	8600 1950 8600 3050
+Wire Wire Line
+	7100 2650 6800 2650
+Wire Wire Line
+	8350 1850 8700 1850
+Wire Wire Line
+	6350 2150 6350 1850
+Connection ~ 6350 2150
+Wire Wire Line
+	6250 2050 6250 1950
+Wire Wire Line
+	6250 1950 6650 1950
+Wire Wire Line
+	6650 2250 6350 2250
+Wire Wire Line
+	6350 2150 6350 2250
+Wire Wire Line
+	6350 2250 6350 2450
+Connection ~ 6350 2250
+Wire Wire Line
+	8200 3050 8600 3050
+Wire Wire Line
+	8350 2950 8350 1850
+Connection ~ 7600 1550
+Wire Wire Line
+	6350 1550 7300 1550
+Connection ~ 7300 1550
+Wire Wire Line
+	7400 1550 7300 1550
+Connection ~ 7400 1550
+Wire Wire Line
+	7400 1550 7500 1550
+Wire Wire Line
+	7600 1550 7500 1550
+Connection ~ 7500 1550
+Wire Wire Line
+	7600 1550 7700 1550
+Wire Wire Line
+	7700 1550 8700 1550
+Connection ~ 7700 1550
 $Comp
 L dk_Interface-Controllers:FT232RL-REEL U2
@@
 $EndComp
 Wire Wire Line
-	7300 3550 7700 3550
-Wire Wire Line
-	6350 1550 7300 1550
-Wire Wire Line
-	7700 1550 9000 1550
-Wire Wire Line
-	5750 3950 5750 3600
-Wire Wire Line
-	8300 3950 8300 2650
-Wire Wire Line
-	8300 2650 8200 2650
-Wire Wire Line
-	5750 3950 8300 3950
-Wire Wire Line
-	7100 2650 6800 2650
-Wire Wire Line
-	6800 2650 6800 3800
-Wire Wire Line
-	7600 3250 7700 3250
-Wire Wire Line
-	7600 3250 7300 3250
-Wire Wire Line
-	7300 3250 7300 3550
-Connection ~ 7600 3250
-Wire Wire Line
-	8200 2950 8350 2950
-Wire Wire Line
-	8350 2950 8350 1850
-Wire Wire Line
-	8350 1850 8700 1850
-Wire Wire Line
-	8200 3050 8600 3050
-Wire Wire Line
-	8600 1950 8600 3050
-Wire Wire Line
-	7600 1550 7700 1550
-Connection ~ 7700 1550
-Wire Wire Line
-	7600 1550 7500 1550
-Connection ~ 7600 1550
-Wire Wire Line
-	7400 1550 7300 1550
-Connection ~ 7300 1550
-Wire Wire Line
-	7400 1550 7500 1550
-Connection ~ 7400 1550
-Connection ~ 7500 1550
-Wire Wire Line
-	3600 1550 5400 1550
-Wire Wire Line
-	6050 6050 4850 6050
-Wire Wire Line
-	4850 6050 4850 6100
-Wire Wire Line
-	4850 6100 4650 6100
+	8700 2350 8950 2350
+Wire Wire Line
+	8950 2350 8950 3850
+Connection ~ 8950 2350
+Wire Wire Line
+	8950 2350 9500 2350
+Wire Wire Line
+	7600 3250 7600 3550
+Wire Wire Line
+	7600 3550 7700 3550
+Wire Wire Line
+	7700 3250 7700 3400
+Wire Wire Line
+	7700 3400 7300 3400
+Wire Wire Line
+	7300 3400 7300 3550
+Connection ~ 7300 3550
+$Comp
+L Device:CP C6
+U 1 1 5F892FD8
+P 8700 1400
+F 0 "C6" H 8500 1450 50  0000 L CNN
+F 1 "10uF" H 8400 1350 50  0000 L CNN
+F 2 "Capacitor_SMD:CP_Elec_3x5.3" H 8738 1250 50  0001 C CNN
+F 3 "~" H 8700 1400 50  0001 C CNN
+	1    8700 1400
+	1    0    0    -1
+$EndComp
+Connection ~ 8700 1550
+Wire Wire Line
+	8700 1550 9000 1550
+Wire Wire Line
+	9000 1250 8700 1250
+Connection ~ 9000 1250
+$Comp
+L Device:LED D1
+U 1 1 5F89779A
+P 7900 1250
+F 0 "D1" V 7939 1133 50  0000 R CNN
+F 1 "LED" V 7848 1133 50  0000 R CNN
+F 2 "LED_SMD:LED_0201_0603Metric" H 7900 1250 50  0001 C CNN
+F 3 "~" H 7900 1250 50  0001 C CNN
+	1    7900 1250
+	0    -1   -1   0
+$EndComp
+$Comp
+L Device:LED D2
+U 1 1 5F8A1CB3
+P 8300 1250
+F 0 "D2" V 8339 1133 50  0000 R CNN
+F 1 "LED" V 8248 1133 50  0000 R CNN
+F 2 "LED_SMD:LED_0201_0603Metric" H 8300 1250 50  0001 C CNN
+F 3 "~" H 8300 1250 50  0001 C CNN
+	1    8300 1250
+	0    -1   -1   0
+$EndComp
+Wire Wire Line
+	8300 1850 8200 1850
+Wire Wire Line
+	7900 1400 8200 1400
+Wire Wire Line
+	8200 1400 8200 1750
+Wire Wire Line
+	8300 1400 8300 1850
+$Comp
+L Device:R R3
+U 1 1 5F8AF9D1
+P 7900 950
+F 0 "R3" H 7970 996 50  0000 L CNN
+F 1 "1kΩ" H 7970 905 50  0000 L CNN
+F 2 "Resistor_SMD:R_0201_0603Metric" V 7830 950 50  0001 C CNN
+F 3 "~" H 7900 950 50  0001 C CNN
+	1    7900 950
+	1    0    0    -1
+$EndComp
+$Comp
+L Device:R R4
+U 1 1 5F8B0311
+P 8300 950
+F 0 "R4" H 8370 996 50  0000 L CNN
+F 1 "1kΩ" H 8370 905 50  0000 L CNN
+F 2 "Resistor_SMD:R_0201_0603Metric" V 8230 950 50  0001 C CNN
+F 3 "~" H 8300 950 50  0001 C CNN
+	1    8300 950
+	1    0    0    -1
+$EndComp
+Wire Wire Line
+	7900 800  8300 800
+Wire Wire Line
+	8300 800  9000 800
+Wire Wire Line
+	9000 800  9000 1250
+Connection ~ 8300 800
 $EndSCHEMATC

Commit message: some fixes not done yet
Parts:
- removed C6: 10uF, Capacitor_SMD:CP_Elec_3x5.3, symbol Device:CP
- added C6: 10uF, Capacitor_SMD:C_0805_2012Metric, symbol Device:C
- C1, C2, C3, C4, C5: footprint Capacitor_SMD:C_0201_0603Metric -> Capacitor_SMD:C_0805_2012Metric
- D1, D2: footprint LED_SMD:LED_0201_0603Metric -> LED_SMD:LED_0805_2012Metric
- L1: footprint Inductor_SMD:L_0201_0603Metric -> Inductor_SMD:L_0805_2012Metric
- R1, R2, R3, R4: footprint Resistor_SMD:R_0201_0603Metric -> Resistor_SMD:R_0805_2012Metric
Connections:
- net GND: now also C6.2
- net at C5.1, J1.1 (VBUS), R3.1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: now also C6.1
Changed lines of the file:
@@
 F 0 "C1" V 4002 2300 50  0000 C CNN
 F 1 "4.7µF" V 3911 2300 50  0000 C CNN
-F 2 "Capacitor_SMD:C_0201_0603Metric" H 3788 2150 50  0001 C CNN
+F 2 "Capacitor_SMD:C_0805_2012Metric" H 3788 2150 50  0001 C CNN
 F 3 "~" H 3750 2300 50  0001 C CNN
 	1    3750 2300
@@
 F 0 "R1" H 6020 3446 50  0000 L CNN
 F 1 "10kΩ" H 6020 3355 50  0000 L CNN
-F 2 "Resistor_SMD:R_0201_0603Metric" V 5880 3400 50  0001 C CNN
+F 2 "Resistor_SMD:R_0805_2012Metric" V 5880 3400 50  0001 C CNN
 F 3 "~" H 5950 3400 50  0001 C CNN
 	1    5950 3400
@@
 F 0 "C2" V 5652 1700 50  0000 C CNN
 F 1 "10µF" V 5561 1700 50  0000 C CNN
-F 2 "Capacitor_SMD:C_0201_0603Metric" H 5438 1550 50  0001 C CNN
+F 2 "Capacitor_SMD:C_0805_2012Metric" H 5438 1550 50  0001 C CNN
 F 3 "~" H 5400 1700 50  0001 C CNN
 	1    5400 1700
@@
 F 0 "L1" H 5452 2046 50  0000 L CNN
 F 1 "2.2µH" H 5452 1955 50  0000 L CNN
-F 2 "Inductor_SMD:L_0201_0603Metric" H 5400 2000 50  0001 C CNN
+F 2 "Inductor_SMD:L_0805_2012Metric" H 5400 2000 50  0001 C CNN
 F 3 "~" H 5400 2000 50  0001 C CNN
 	1    5400 2000
@@
 F 0 "C3" V 6602 1700 50  0000 C CNN
 F 1 "4.7µF" V 6511 1700 50  0000 C CNN
-F 2 "Capacitor_SMD:C_0201_0603Metric" H 6388 1550 50  0001 C CNN
+F 2 "Capacitor_SMD:C_0805_2012Metric" H 6388 1550 50  0001 C CNN
 F 3 "~" H 6350 1700 50  0001 C CNN
 	1    6350 1700
@@
 F 0 "R2" H 6720 2146 50  0000 L CNN
 F 1 "100kΩ" H 6720 2055 50  0000 L CNN
-F 2 "Resistor_SMD:R_0201_0603Metric" V 6580 2100 50  0001 C CNN
+F 2 "Resistor_SMD:R_0805_2012Metric" V 6580 2100 50  0001 C CNN
 F 3 "~" H 6650 2100 50  0001 C CNN
 	1    6650 2100
@@
 F 0 "C4" H 7215 3046 50  0000 L CNN
 F 1 "0.1uF" H 7215 2955 50  0000 L CNN
-F 2 "Capacitor_SMD:C_0201_0603Metric" H 7138 2850 50  0001 C CNN
+F 2 "Capacitor_SMD:C_0805_2012Metric" H 7138 2850 50  0001 C CNN
 F 3 "~" H 7100 3000 50  0001 C CNN
 	1    7100 3000
@@
 F 0 "C5" H 9115 1446 50  0000 L CNN
 F 1 "0.1uF" H 9115 1355 50  0000 L CNN
-F 2 "Capacitor_SMD:C_0201_0603Metric" H 9038 1250 50  0001 C CNN
+F 2 "Capacitor_SMD:C_0805_2012Metric" H 9038 1250 50  0001 C CNN
 F 3 "~" H 9000 1400 50  0001 C CNN
 	1    9000 1400
@@
 Wire Wire Line
 	7600 1550 7700 1550
-Wire Wire Line
-	7700 1550 8700 1550
 Connection ~ 7700 1550
 $Comp
@@
 	7300 3400 7300 3550
 Connection ~ 7300 3550
-$Comp
-L Device:CP C6
-U 1 1 5F892FD8
-P 8700 1400
-F 0 "C6" H 8500 1450 50  0000 L CNN
-F 1 "10uF" H 8400 1350 50  0000 L CNN
-F 2 "Capacitor_SMD:CP_Elec_3x5.3" H 8738 1250 50  0001 C CNN
-F 3 "~" H 8700 1400 50  0001 C CNN
-	1    8700 1400
-	1    0    0    -1
-$EndComp
-Connection ~ 8700 1550
-Wire Wire Line
-	8700 1550 9000 1550
 Wire Wire Line
 	9000 1250 8700 1250
@@
 F 0 "D1" V 7939 1133 50  0000 R CNN
 F 1 "LED" V 7848 1133 50  0000 R CNN
-F 2 "LED_SMD:LED_0201_0603Metric" H 7900 1250 50  0001 C CNN
+F 2 "LED_SMD:LED_0805_2012Metric" H 7900 1250 50  0001 C CNN
 F 3 "~" H 7900 1250 50  0001 C CNN
 	1    7900 1250
@@
 F 0 "D2" V 8339 1133 50  0000 R CNN
 F 1 "LED" V 8248 1133 50  0000 R CNN
-F 2 "LED_SMD:LED_0201_0603Metric" H 8300 1250 50  0001 C CNN
+F 2 "LED_SMD:LED_0805_2012Metric" H 8300 1250 50  0001 C CNN
 F 3 "~" H 8300 1250 50  0001 C CNN
 	1    8300 1250
@@
 F 0 "R3" H 7970 996 50  0000 L CNN
 F 1 "1kΩ" H 7970 905 50  0000 L CNN
-F 2 "Resistor_SMD:R_0201_0603Metric" V 7830 950 50  0001 C CNN
+F 2 "Resistor_SMD:R_0805_2012Metric" V 7830 950 50  0001 C CNN
 F 3 "~" H 7900 950 50  0001 C CNN
 	1    7900 950
@@
 F 0 "R4" H 8370 996 50  0000 L CNN
 F 1 "1kΩ" H 8370 905 50  0000 L CNN
-F 2 "Resistor_SMD:R_0201_0603Metric" V 8230 950 50  0001 C CNN
+F 2 "Resistor_SMD:R_0805_2012Metric" V 8230 950 50  0001 C CNN
 F 3 "~" H 8300 950 50  0001 C CNN
 	1    8300 950
@@
 	9000 800  9000 1250
 Connection ~ 8300 800
+Wire Wire Line
+	7700 1550 8700 1550
+$Comp
+L Device:C C6
+U 1 1 5F8242E5
+P 8700 1400
+F 0 "C6" H 8500 1400 50  0000 L CNN
+F 1 "10uF" H 8500 1300 50  0000 L CNN
+F 2 "Capacitor_SMD:C_0805_2012Metric" H 8738 1250 50  0001 C CNN
+F 3 "~" H 8700 1400 50  0001 C CNN
+	1    8700 1400
+	1    0    0    -1
+$EndComp
+Connection ~ 8700 1550
+Wire Wire Line
+	8700 1550 9000 1550
 $EndSCHEMATC
