File: pcb/ece477.kicad_pcb (KiCad board)
At the start: 2 copper layers, 48.2 x 40 mm, 27 parts, among them J1 USB_B, Q1 MMBT2222, Q2 MMBT2222, SW1 SW_DIP_x01, U1 ESP32-WROOM-32, U2 FT232RL-REEL, U3 LM3671, U4 ADA254, U5 ADA751

Commit message: pcb final touch
Routing:
- net GND: vias 10 -> 11
Changed lines of the file:
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@@
     (thickness 1.6)
     (drawings 24)
-    (tracks 273)
+    (tracks 274)
     (zones 0)
     (modules 27)
@@
   (via (at 171.2 84) (size 0.8) (drill 0.4) (layers F.Cu B.Cu) (net 1))
   (via (at 173 79.75) (size 0.8) (drill 0.4) (layers F.Cu B.Cu) (net 1))
-  (segment (start 163.055 89.5) (end 163.055 90.265002) (width 0.25) (layer F.Cu) (net 64))
   (via (at 171.2 83) (size 0.8) (drill 0.4) (layers F.Cu B.Cu) (net 1))
   (via (at 148.4 86.2) (size 0.8) (drill 0.4) (layers F.Cu B.Cu) (net 1))
@@
   (segment (start 178.55 94.35) (end 177.4 93.2) (width 0.25) (layer F.Cu) (net 1))
   (segment (start 181.04 94.35) (end 178.55 94.35) (width 0.25) (layer F.Cu) (net 1))
+  (via (at 166.6 112) (size 0.8) (drill 0.4) (layers F.Cu B.Cu) (net 1))
   (segment (start 160.05 86.75) (end 157.8 84.5) (width 0.4) (layer F.Cu) (net 2))
   (segment (start 178.2625 85) (end 178.2 85.0625) (width 0.4) (layer F.Cu) (net 2))
@@
   (segment (start 143.8 82.2625) (end 145.6 84.0625) (width 0.25) (layer F.Cu) (net 63))
   (segment (start 143.8 80.9375) (end 143.8 82.2625) (width 0.25) (layer F.Cu) (net 63))
+  (segment (start 163.055 89.5) (end 163.055 90.265002) (width 0.25) (layer F.Cu) (net 64))
   (segment (start 168.6 98.65) (end 168.6 99.55) (width 0.25) (layer F.Cu) (net 64))
   (segment (start 165.635002 89.5) (end 168.6 92.464998) (width 0.25) (layer F.Cu) (net 64))
