File: pcb/ece477.kicad_pcb (KiCad board)
At the start: 2 copper layers, 48.2 x 40 mm, 27 parts, among them J1 USB_B, Q1 MMBT2222, Q2 MMBT2222, SW1 SW_DIP_x01, U1 ESP32-WROOM-32, U2 FT232RL-REEL, U3 LM3671, U4 ADA254, U5 ADA751

Commit message: added uart cmd
Other:
- board text added: "JLCJLCJLCJLC"
- board text removed: "Fingerprint scanner"
Changed lines of the file:
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@@
   (general
     (thickness 1.6)
-    (drawings 24)
+    (drawings 20)
     (tracks 274)
     (zones 0)
@@
     (visible_elements FFFDFF7F)
     (pcbplotparams
-      (layerselection 0x010fc_ffffffff)
+      (layerselection 0x3ffff_ffffffff)
       (usegerberextensions false)
       (usegerberattributes false)
@@
     )
   )
+  (gr_text JLCJLCJLCJLC (at 139.4 81.4 90) (layer B.SilkS)
+    (effects (font (size 1 1) (thickness 0.15)) (justify mirror))
+  )
   (gr_line (start 139.8 115) (end 144 115) (layer Edge.Cuts) (width 0.05))
   (gr_line (start 139.8 75) (end 144 75) (layer Edge.Cuts) (width 0.05))
@@
   )
   (gr_line (start 182 115) (end 144 115) (layer Edge.Cuts) (width 0.05))
-  (gr_text "Fingerprint scanner" (at 165 63) (layer F.Paste)
-    (effects (font (size 1 1) (thickness 0.15)))
-  )
-  (gr_line (start 137 53) (end 137 73) (layer F.Paste) (width 0.15))
-  (gr_line (start 193 53) (end 137 53) (layer F.Paste) (width 0.15))
-  (gr_line (start 193 73) (end 193 53) (layer F.Paste) (width 0.15))
-  (gr_line (start 137 73) (end 193 73) (layer F.Paste) (width 0.15))
   (gr_line (start 136.8 112) (end 136.8 78) (layer Edge.Cuts) (width 0.05))
   (gr_line (start 185 78) (end 185 112) (layer Edge.Cuts) (width 0.05))

Commit message: added function description
Other:
- board text removed: "FB"
Changed lines of the file:
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@@
   (general
     (thickness 1.6)
-    (drawings 20)
+    (drawings 19)
     (tracks 274)
     (zones 0)
@@
     (effects (font (size 0.75 0.75) (thickness 0.1)))
   )
-  (gr_text FB (at 161.4 82.6) (layer F.SilkS)
-    (effects (font (size 0.75 0.75) (thickness 0.1)))
-  )
